File: hw/coral-ir.kicad_pcb (KiCad board)
At the start: 2 copper layers, 35 x 55 mm, 28 parts, among them IC1 ESP32-C6-WROOM-1-N8, IC2 TPS74633PQWDRBRQ1, J1 USB4105-GF-A, Q1 MMSS8050HE3-H-TP

Commit message: Finished revision 1, ready for production
Parts:
- added R9: 1k, PCBLib:R_Vishay_CRCW_0402, F.Cu at (108.5, 56.0)
- added S1: SLW-1678105-6A-N-D, PCBLib:SLW16781056AND, B.Cu at (115.3, 58.1)
- added S2: TL3305AF260QG, PCBLib:TL3305AF160QG, F.Cu at (110.5, 50.3)
- Q1: value MMSS8050HE3-H-TP -> FMMT619TA; footprint PCBLib:SOT-23 -> PCBLib:SOT95P237X112-3N
- moved BT1 5.22 mm to (102.5, 66.5)
- moved D1 3.72 mm to (117.7, 74.6), turned to 90 degrees
- moved D4 3.65 mm to (115.7, 72.9), turned to -90 degrees
- moved D2 1.92 mm to (113.8, 70.7), turned to 180 degrees
- moved C3 1.20 mm to (115.3, 74.8), turned to 0 degrees
Connections:
- BT1 pad P: +5V -> +3V
- C3 pad 1: +5V -> VBUS
- IC1 pad 15: unconnected-(IC1-IO9-Pad15) -> RESET
- IC2 pad 5: +5V -> VBUS
- IC2 pad 8: +5V -> VBUS
Routing:
- net VBUS: track 0.00 -> 34.9 mm, vias 0 -> 1
- net +3V: track 0.00 -> 20.1 mm
- net +5V: track 39.4 -> 21.6 mm, vias 1 -> 0
- net Net-(S2-A1): track 0.00 -> 9.35 mm
- net RESET: track 0.00 -> 2.70 mm
- net IR: track 35.8 -> 37.9 mm
- net +3V3: track 44.3 -> 45.6 mm
- net Earth: track 10.1 -> 9.26 mm, vias 9 -> 8
- net USB_DP: track 25.0 -> 24.4 mm
- net USB_DN: track 24.7 -> 24.1 mm
