File: hw/coral-ir.kicad_sch (KiCad schematic)
At the start: 28 parts, among them IC1 ESP32-C6-WROOM-1-N8, IC2 TPS74633PQWDRBRQ1, J1 USB4105-GF-A, Q1 MMSS8050HE3-H-TP

Commit message: Finished revision 1, ready for production
Parts:
- removed Q1: MMSS8050HE3-H-TP, PCBLib:SOT-23, symbol PCBLib:SS8050
- added Q1: FMMT619TA, PCBLib:SOT95P237X112-3N, symbol PCBLib:FMMT619TA
- added R9: 1k, PCBLib:R_Vishay_CRCW_0402, symbol Device:R_Small
- added S1: SLW-1678105-6A-N-D, PCBLib:SLW16781056AND, symbol PCBLib:SLW-1678105-6A-N-D
- added S2: TL3305AF260QG, PCBLib:TL3305AF160QG, symbol PCBLib:TL3305AF260QG
Connections:
- net +5V: now also S1.1 (NC_1), S1.6 (NC_2); no longer BT1.P, C3.1, IC2.5 (EN), IC2.8 (IN)
- net Earth: now also Q1.2 (E), S2.3 (B1), S2.4 (B2)
- net RESET: now reaches IC1.15 (IO9)
- net RESET: now also R9.2
- net at R5.1, R6.1: now also Q1.1 (B)
- net at D5.C, D6.C: now also Q1.3 (C)
- new net: R9.1, S2.1 (A1), S2.2 (A2)
- new net +3V: BT1.P, S1.3 (NO_1), S1.4 (NO_2)
- new net VBUS: C3.1, IC2.5 (EN), IC2.8 (IN), S1.2 (COM_1), S1.5 (COM_2)
- no-connect marks 30 -> 29
Other:
- note added: "Power Switch"
- note added: "Reset Button"
- note added: "V_{BE(sat)} = 0.9 V I_{B} = 2.4 mA = (3.3 V - V_{BE(sat)}) / R_{5} R_{5} = 1kΩ"
- note added: "V_{F} = 2.5 V V_{CE(sat)} = 100 mV V_{R} = 3.3 V - V_{F} - V_{CE(sat)} = 0.7 V I_{F} = 179 mA = V_{R} / R_{7,8} R_{7,8} = 3.92 Ω"
- note removed: "204 mA = 0.8 V / 3.92 Ohm"
- note removed: "I_B = 2.6 mA = (3.3 V - 0.7 V) / 1kOhm"
- moved on the sheet: BT1, D5, D6, R5, R6, R7, R8
